Commit message: added the mesh file and decreased the size of the cameras

File: spiri_description/sensors/generic_camera.urdf.xacro (robot description, xacro)
@@ -17,5 +17,5 @@
         <origin xyz="0 0 0" rpy="0 0 0" />
         <geometry>
-          <box size="0.01 0.01 0.01" />
+          <box size="0.001 0.001 0.001" />
         </geometry>
         <material name="Blue">
@@ -26,5 +26,5 @@
         <origin xyz="0 0 0" rpy="0 0 0" />
         <geometry>
-          <box size="0.01 0.01 0.01" />
+          <box size="0.001 0.001 0.001" />
         </geometry>
       </collision>

File: spiri_description/sensors/tof.urdf.xacro (robot description, xacro)
@@ -17,5 +17,5 @@
         <origin xyz="0 0 0" rpy="0 0 0" />
         <geometry>
-          <box size="0.01 0.01 0.01" />
+          <box size="0.001 0.001 0.001" />
         </geometry>
         <material name="Blue">
@@ -26,5 +26,5 @@
         <origin xyz="0 0 0" rpy="0 0 0" />
         <geometry>
-          <box size="0.01 0.01 0.01" />
+          <box size="0.001 0.001 0.001" />
         </geometry>
       </collision>

File: spiri_description/urdf/spiri_base.urdf.xacro (robot description, xacro)
@@ -20,8 +20,8 @@
       <origin
         xyz="0 0 0"
-        rpy="0 0 0" />
+        rpy="1.57 0 0" />
       <geometry>
         <mesh
-          filename="package://spiri_description/meshes/base_link.STL" />
+          filename="package://spiri_description/meshes/spiri.dae" />
       </geometry>
     </visual>
