Commit message: added pcl2 by uisng kinect as a replacement for tof

File: spiri_description/sensors/quadrotor_sensors.gazebo.xacro (robot description, xacro)
@@ -63,7 +63,7 @@
     </xacro:generic_camera>
 <!-- TOF camera -->
- <xacro:include filename="$(find spiri_description)/sensors/tof.urdf.xacro" />
-    <xacro:generic_tof name="tof" parent="forward_cam_link" ros_topic="tof" update_rate="20" noise="0.0">
-      <origin xyz="0.00 -0.01 0.00" rpy="${M_PI/2} 0 0"/>
-    </xacro:generic_tof>
+ <xacro:include filename="$(find spiri_description)/sensors/tof_kinect.urdf.xacro" />
+     <xacro:kinect_camera name="camera" parent="base_link">
+      <origin xyz="-0.04 -0.00 0.1" rpy="0 0 ${M_PI}"/>
+    </xacro:kinect_camera>
 </robot>

File: spiri_description/sensors/tof.urdf.xacro (robot description, xacro)
@@ -2,5 +2,5 @@
 <robot xmlns:xacro="http://ros.org/wiki/xacro">
   <xacro:property name="M_PI" value="3.1415926535897931" />
-  <xacro:macro name="generic_tof" params="name parent *origin ros_topic noise update_rate">
+  <xacro:macro name="generic_tof" params="name parent *origin ros_topic noise update_rate camera_name">
     <joint name="${name}_joint" type="fixed">
       <xacro:insert_block name="origin" />

Commit message: added pcl2 for block laser, even reduced the horizontal samples (lag)

File: spiri_description/sensors/quadrotor_sensors.gazebo.xacro (robot description, xacro)
@@ -54,5 +54,5 @@
     <!-- Downward facing camera -->
     <xacro:include filename="$(find spiri_description)/sensors/generic_camera.urdf.xacro" />
-    <xacro:generic_camera name="downward_cam" parent="base_link" ros_topic="camera/image" cam_info_topic="camera/camera_info" update_rate="20" res_x="640" res_y="480" image_format="R8G8B8" hfov="65">
+    <xacro:generic_camera name="downward_cam" parent="base_link" ros_topic="camera/image" cam_info_topic="camera/camera_info" update_rate="30" res_x="640" res_y="480" image_format="R8G8B8" hfov="65">
       <origin xyz="-0.04 0.0 -0.035" rpy="0 ${M_PI/2} 0"/>
  </xacro:generic_camera>
@@ -63,7 +63,11 @@
     </xacro:generic_camera>
 <!-- TOF camera -->
- <xacro:include filename="$(find spiri_description)/sensors/tof_kinect.urdf.xacro" />
+ <!--xacro:include filename="$(find spiri_description)/sensors/tof_kinect.urdf.xacro" />
      <xacro:kinect_camera name="camera" parent="base_link">
       <origin xyz="-0.04 -0.00 0.1" rpy="0 0 ${M_PI}"/>
-    </xacro:kinect_camera>
+    </xacro:kinect_camera-->
+ <xacro:include filename="$(find spiri_description)/sensors/tof.urdf.xacro" />
+    <xacro:generic_tof name="tof" parent="forward_cam_link" ros_topic="tof" update_rate="30" noise="0.0">
+      <origin xyz="0.00 -0.01 0.00" rpy="${M_PI/2} 0 0"/>
+    </xacro:generic_tof>
 </robot>

File: spiri_description/sensors/tof.urdf.xacro (robot description, xacro)
@@ -2,5 +2,5 @@
 <robot xmlns:xacro="http://ros.org/wiki/xacro">
   <xacro:property name="M_PI" value="3.1415926535897931" />
-  <xacro:macro name="generic_tof" params="name parent *origin ros_topic noise update_rate camera_name">
+  <xacro:macro name="generic_tof" params="name parent *origin ros_topic noise update_rate">
     <joint name="${name}_joint" type="fixed">
       <xacro:insert_block name="origin" />
@@ -36,5 +36,5 @@
 	  <scan>
           <horizontal>
-		<samples>300</samples>
+		<samples>100</samples>
 		<resolution>1.0</resolution>
 		<min_angle>-0.5236</min_angle>
@@ -54,5 +54,5 @@
 	  </range>
 	</ray>
-        <plugin name="${name}_tof_controller" filename="libgazebo_ros_block_laser.so">
+        <plugin name="${name}_tof_controller" filename="libgazebo_block_laser_pcl2.so">
           <topicName>${ros_topic}</topicName>
           <alwaysOn>true</alwaysOn>

File: spiri_description/sensors/tof_depth.urdf.xacro (robot description, xacro)
@@ -1,70 +1,96 @@
 <?xml version="1.0"?>
 <robot xmlns:xacro="http://ros.org/wiki/xacro">
-  <xacro:property name="M_PI" value="3.1415926535897931" />
-  <xacro:macro name="generic_tof" params="name parent *origin ros_topic noise update_rate camera_name">
-    <joint name="${name}_joint" type="fixed">
-      <xacro:insert_block name="origin" />
-      <parent link="${parent}"/>
-      <child link="${name}_link"/>
-    </joint>
-    <link name="${name}_link">
-      <inertial>
-        <mass value="0.001" />
-        <origin xyz="0 0 0" rpy="0 0 0" />
-        <inertia ixx="0.0001" ixy="0" ixz="0" iyy="0.0001" iyz="0" izz="0.0001" />
-      </inertial>
-      <visual>
-        <origin xyz="0 0 0" rpy="0 0 0" />
-        <geometry>
+    <xacro:property name="M_PI" value="3.1415926535897931" />
+    <xacro:macro name="kinect_camera_model" params="name parent *origin">
+      <joint name="${name}_joint" type="fixed">
+        <xacro:insert_block name="origin" />
+        <parent link="${parent}"/>
+        <child link="${name}_link"/>
+      </joint>
+      <link name="${name}_link">
+        <inertial_sphere mass="0.01" diameter="0.07" />
+        <visual>
+          <origin xyz="0 0 0" rpy="0 0 0" />
+          <geometry>
           <box size="0.01 0.01 0.01" />
         </geometry>
-        <material name="Blue">
+<material name="Blue">
           <color rgba="0.0 0.0 0.8 1"/>
         </material>
-      </visual>
-      <collision>
-        <origin xyz="0 0 0" rpy="0 0 0" />
-        <geometry>
+        </visual>
+        <collision>
+          <origin xyz="0 0 0" rpy="0 0 0" />
+          <geometry>
           <box size="0.01 0.01 0.01" />
         </geometry>
-      </collision>
-    </link>
-   <gazebo reference="${name}_link">
-   <sensor type="depth" name="depth_camera">
-        <always_on>1</always_on>
-        <visualize>true</visualize>
-<topic>tof</topic>
-        <camera>
-            <horizontal_fov>1.047</horizontal_fov>
+        </collision>
+      </link>
+      <joint name="${name}_depth_joint" type="fixed">
+        <origin xyz="0.0 -0.02 0.0" rpy="0 0 0" />
+        <parent link="${name}_link" />
+        <child link="${name}_depth_frame"/>
+      </joint>
+      <link name="${name}_depth_frame"/>
+      <joint name="${name}_depth_optical_joint" type="fixed">
+        <origin xyz="0 0 0" rpy="${-M_PI/2} 0.0 ${-M_PI/2}" />
+        <parent link="${name}_depth_frame" />
+        <child link="${name}_depth_optical_frame"/>
+      </joint>
+      <link name="${name}_depth_optical_frame"/>
+      <joint name="${name}_rgb_joint" type="fixed">
+        <origin xyz="0.0 -0.0125 0.0" rpy="0 0 0" />
+        <parent link="${name}_link" />
+        <child link="${name}_rgb_frame"/>
+      </joint>
+      <link name="${name}_rgb_frame"/>
+      <joint name="${name}_rgb_optical_joint" type="fixed">
+        <origin xyz="0 0 0" rpy="${-M_PI/2} 0.0 ${-M_PI/2}" />
+        <parent link="${name}_rgb_frame" />
+        <child link="${name}_rgb_optical_frame"/>
+      </joint>
+      <link name="${name}_rgb_optical_frame"/>
+    </xacro:macro>
+    <xacro:macro name="kinect_camera" params="name parent *origin">
+      <xacro:kinect_camera_model name="${name}" parent="${parent}">
+        <xacro:insert_block name="origin" />
+      </xacro:kinect_camera_model>
+      <gazebo reference="${name}_depth_frame">
+        <sensor type="depth" name="${name}">
+          <update_rate>30</update_rate>
+          <camera>
+            <horizontal_fov>1.407</horizontal_fov>
             <image>
-                <width>640</width>
-                <height>480</height>
-                <format>R8G8B8</format>
+              <format>R8G8B8</format>
+              <width>640</width>
+              <height>480</height>
             </image>
-            <depth_camera>
-            </depth_camera>
             <clip>
-                <near>0.02</near>
-                <far>300</far>
+              <near>1.0</near>
+              <far>3</far>
             </clip>
-        </camera>
-        <plugin name="camera_controller" filename="libDepthCameraPlugin.so">
-        <alwaysOn>true</alwaysOn>
-                <updateRate>10.0</updateRate>
-                <cameraName>depth_cam</cameraName>
-                <frameName>openni_camera_link</frameName>
-                <hackBaseline>0.07</hackBaseline>
-                <distortionK1>0.0</distortionK1>
-                <distortionK2>0.0</distortionK2>
-                <distortionK3>0.0</distortionK3>
-                <distortionT1>0.0</distortionT1>
-                <distortionT2>0.0</distortionT2>
-            <CxPrime>0.0</CxPrime>
-            <Cx>0.0</Cx>
-            <Cy>0.0</Cy>
-            <focalLength>0.0</focalLength>
-  </plugin>
-    </sensor>
-    </gazebo>
-  </xacro:macro>
-</robot>
+          </camera>
+          <plugin name="${name}_camera_controller" filename="libDepthCameraPlugin.so">
+	<baseline>0.2</baseline>
+	<alwaysOn>true</alwaysOn>
+            <updateRate>20</updateRate>
+            <imageTopicName>${name}/rgb/image_raw</imageTopicName>
+            <depthImageTopicName>${name}/depth/image_raw</depthImageTopicName>
+            <depthImageCameraInfoTopicName>${name}/depth/camera_info</depthImageCameraInfoTopicName>
+            <pointCloudTopicName>${name}/depth/points</pointCloudTopicName>
+            <frameName>${name}_depth_optical_frame</frameName>
+   <distortionK1>0.00000001</distortionK1>
+    <distortionK2>0.00000001</distortionK2>
+    <distortionK3>0.00000001</distortionK3>
+    <distortionT1>0.00000001</distortionT1>
+    <distortionT2>0.00000001</distortionT2>
+	     <pointCloudCutoff>0.5</pointCloudCutoff>
+  <CxPrime>0</CxPrime>
+    <Cx>0</Cx>
+    <Cy>0</Cy>
+    <focalLength>0</focalLength>
+    <hackBaseline>0</hackBaseline>
+          </plugin>
+        </sensor>
+      </gazebo>
+    </xacro:macro>
+  </robot>

File: spiri_description/sensors/tof_kinect.urdf.xacro (robot description, xacro)
@@ -57,7 +57,7 @@
       <gazebo reference="${name}_depth_frame">
         <sensor type="depth" name="${name}">
-          <update_rate>20</update_rate>
+          <update_rate>30</update_rate>
           <camera>
-            <horizontal_fov>${60 * M_PI/180.0}</horizontal_fov>
+            <horizontal_fov>1.407</horizontal_fov>
             <image>
               <format>R8G8B8</format>
@@ -66,10 +66,11 @@
             </image>
             <clip>
-              <near>0.05</near>
+              <near>1.0</near>
               <far>3</far>
             </clip>
           </camera>
           <plugin name="${name}_camera_controller" filename="libgazebo_ros_openni_kinect.so">
-            <alwaysOn>true</alwaysOn>
+	<baseline>0.2</baseline>
+	<alwaysOn>true</alwaysOn>
             <updateRate>20</updateRate>
             <imageTopicName>${name}/rgb/image_raw</imageTopicName>
@@ -79,9 +80,15 @@
             <pointCloudTopicName>${name}/depth/points</pointCloudTopicName>
             <frameName>${name}_depth_optical_frame</frameName>
-            <distortion_k1>0.0</distortion_k1>
-            <distortion_k2>0.0</distortion_k2>
-            <distortion_k3>0.0</distortion_k3>
-            <distortion_t1>0.0</distortion_t1>
-            <distortion_t2>0.0</distortion_t2>
+   <distortionK1>0.00000001</distortionK1>
+    <distortionK2>0.00000001</distortionK2>
+    <distortionK3>0.00000001</distortionK3>
+    <distortionT1>0.00000001</distortionT1>
+    <distortionT2>0.00000001</distortionT2>
+	     <pointCloudCutoff>0.5</pointCloudCutoff>
+  <CxPrime>0</CxPrime>
+    <Cx>0</Cx>
+    <Cy>0</Cy>
+    <focalLength>0</focalLength>
+    <hackBaseline>0</hackBaseline>
           </plugin>
         </sensor>

Commit message: goal can be sent by script and we can get the feedback(state, goal status) as well

File: spiri_description/sensors/quadrotor_sensors.gazebo.xacro (robot description, xacro)
@@ -69,5 +69,5 @@
  <xacro:include filename="$(find spiri_description)/sensors/tof.urdf.xacro" />
     <xacro:generic_tof name="tof" parent="forward_cam_link" ros_topic="tof" update_rate="30" noise="0.0">
-      <origin xyz="0.00 -0.01 0.00" rpy="${M_PI/2} 0 0"/>
+      <origin xyz="0.00 0.02 0.0" rpy="${M_PI/2} 0 0"/>
     </xacro:generic_tof>
 </robot>

File: spiri_description/sensors/tof.urdf.xacro (robot description, xacro)
@@ -58,5 +58,5 @@
           <alwaysOn>true</alwaysOn>
           <updateRate>${update_rate}</updateRate>
-          <pcl>1.0</pcl>
+          <pcl>2.0</pcl>
 	  <gaussianNoise>${noise}</gaussianNoise>
           <frameName>${name}_link</frameName>

Commit message: added ony big launch file for launching moveit, gazebo and action_controller

File: spiri_description/sensors/quadrotor_sensors.gazebo.xacro (robot description, xacro)
@@ -60,5 +60,5 @@
     <xacro:include filename="$(find spiri_description)/sensors/generic_camera.urdf.xacro" />
     <xacro:generic_camera name="forward_cam" parent="base_link" ros_topic="camera/image" cam_info_topic="camera/camera_info" update_rate="30" res_x="1920" res_y="1080" image_format="R8G8B8" hfov="67.3">
-      <origin xyz="-0.04 0.0 0.02" rpy="${M_PI/2} 0 ${M_PI}"/>
+      <origin xyz="-0.04 0.0 0.05" rpy="0 0 ${M_PI}"/>
     </xacro:generic_camera>
 <!-- TOF camera -->
@@ -69,5 +69,5 @@
  <xacro:include filename="$(find spiri_description)/sensors/tof.urdf.xacro" />
     <xacro:generic_tof name="tof" parent="forward_cam_link" ros_topic="tof" update_rate="30" noise="0.0">
-      <origin xyz="0.00 0.02 0.0" rpy="${M_PI/2} 0 0"/>
+      <origin xyz="0.00 0.0 0.02" rpy="${M_PI} 0 0"/>
     </xacro:generic_tof>
 </robot>

Commit message: cameras are placed and the front camera is rotated by 90

File: spiri_description/sensors/quadrotor_sensors.gazebo.xacro (robot description, xacro)
@@ -60,5 +60,5 @@
     <xacro:include filename="$(find spiri_description)/sensors/generic_camera.urdf.xacro" />
     <xacro:generic_camera name="forward_cam" parent="base_link" ros_topic="camera/image" cam_info_topic="camera/camera_info" update_rate="30" res_x="1920" res_y="1080" image_format="R8G8B8" hfov="67.3">
-      <origin xyz="-0.04 0.0 0.05" rpy="0 0 ${M_PI}"/>
+      <origin xyz="-0.04 0.005 0.01" rpy="${M_PI/2} 0 ${M_PI}"/>
     </xacro:generic_camera>
 <!-- TOF camera -->
@@ -69,5 +69,5 @@
  <xacro:include filename="$(find spiri_description)/sensors/tof.urdf.xacro" />
     <xacro:generic_tof name="tof" parent="forward_cam_link" ros_topic="tof" update_rate="30" noise="0.0">
-      <origin xyz="0.00 0.0 0.02" rpy="${M_PI} 0 0"/>
+      <origin xyz="0.00 0.0 -0.01" rpy="${3*M_PI/2} 0 0"/>
     </xacro:generic_tof>
 </robot>

Commit message: changed the settings of camera and added a ground plane

File: spiri_description/sensors/quadrotor_sensors.gazebo.xacro (robot description, xacro)
@@ -60,5 +60,5 @@
     <xacro:include filename="$(find spiri_description)/sensors/generic_camera.urdf.xacro" />
     <xacro:generic_camera name="forward_cam" parent="base_link" ros_topic="camera/image" cam_info_topic="camera/camera_info" update_rate="30" res_x="1920" res_y="1080" image_format="R8G8B8" hfov="67.3">
-      <origin xyz="-0.04 0.005 0.01" rpy="${M_PI/2} 0 ${M_PI}"/>
+      <origin xyz="-0.04 0.0 0.05" rpy="0 0 ${M_PI}"/>
     </xacro:generic_camera>
 <!-- TOF camera -->
@@ -69,5 +69,5 @@
  <xacro:include filename="$(find spiri_description)/sensors/tof.urdf.xacro" />
     <xacro:generic_tof name="tof" parent="forward_cam_link" ros_topic="tof" update_rate="30" noise="0.0">
-      <origin xyz="0.00 0.0 -0.01" rpy="${3*M_PI/2} 0 0"/>
+      <origin xyz="0.00 0.0 0.02" rpy="${M_PI} 0 0"/>
     </xacro:generic_tof>
 </robot>

Commit message: changed the camera locations

File: spiri_description/sensors/quadrotor_sensors.gazebo.xacro (robot description, xacro)
@@ -57,8 +57,13 @@
       <origin xyz="-0.04 0.0 -0.035" rpy="0 ${M_PI/2} 0"/>
  </xacro:generic_camera>
-<!-- Forward facing camera -->
+<!-- Left Forward facing camera -->
     <xacro:include filename="$(find spiri_description)/sensors/generic_camera.urdf.xacro" />
-    <xacro:generic_camera name="forward_cam" parent="base_link" ros_topic="camera/image" cam_info_topic="camera/camera_info" update_rate="30" res_x="1920" res_y="1080" image_format="R8G8B8" hfov="67.3">
-      <origin xyz="-0.04 0.0 0.05" rpy="0 0 ${M_PI}"/>
+    <xacro:generic_camera name="left_cam" parent="base_link" ros_topic="camera/image" cam_info_topic="camera/camera_info" update_rate="30" res_x="1920" res_y="1080" image_format="R8G8B8" hfov="67.3">
+      <origin xyz="-0.064 -0.0245 -0.0265" rpy="0 0.17 ${M_PI}"/>
+    </xacro:generic_camera>
+<!-- Right Forward facing camera -->
+    <xacro:include filename="$(find spiri_description)/sensors/generic_camera.urdf.xacro" />
+    <xacro:generic_camera name="right_cam" parent="base_link" ros_topic="camera/image" cam_info_topic="camera/camera_info" update_rate="30" res_x="1920" res_y="1080" image_format="R8G8B8" hfov="67.3">
+      <origin xyz="-0.064 0.0245 -0.0265" rpy="0 0.17 ${M_PI}"/>
     </xacro:generic_camera>
 <!-- TOF camera -->
@@ -67,7 +72,7 @@
       <origin xyz="-0.04 -0.00 0.1" rpy="0 0 ${M_PI}"/>
     </xacro:kinect_camera-->
- <xacro:include filename="$(find spiri_description)/sensors/tof.urdf.xacro" />
+ <!--xacro:include filename="$(find spiri_description)/sensors/tof.urdf.xacro" />
     <xacro:generic_tof name="tof" parent="forward_cam_link" ros_topic="tof" update_rate="30" noise="0.0">
       <origin xyz="0.00 0.0 0.02" rpy="${M_PI} 0 0"/>
-    </xacro:generic_tof>
+    </xacro:generic_tof-->
 </robot>

Commit message: placement of cameras

File: spiri_description/sensors/quadrotor_sensors.gazebo.xacro (robot description, xacro)
@@ -59,11 +59,11 @@
 <!-- Left Forward facing camera -->
     <xacro:include filename="$(find spiri_description)/sensors/generic_camera.urdf.xacro" />
-    <xacro:generic_camera name="stereo/left" parent="base_link" ros_topic="image_raw" cam_info_topic="camera_info" update_rate="30" res_x="320" res_y="240" image_format="R8G8B8" hfov="67.3">
-      <origin xyz="-0.064 -0.0245 -0.0265" rpy="0 0.17 ${M_PI}"/>
+    <xacro:generic_camera name="stereo/left" parent="base_link" ros_topic="image_raw" cam_info_topic="camera_info" update_rate="30" res_x="320" res_y="240" image_format="R8G8B8" hfov="65.0">
+      <origin xyz="-0.064 -0.0245 -0.0265" rpy="0 0.261 ${M_PI}"/>
     </xacro:generic_camera>
 <!-- Right Forward facing camera -->
     <xacro:include filename="$(find spiri_description)/sensors/generic_camera.urdf.xacro" />
-    <xacro:generic_camera name="stereo/right" parent="base_link" ros_topic="image_raw" cam_info_topic="camera_info" update_rate="30" res_x="320" res_y="240" image_format="R8G8B8" hfov="67.3">
-      <origin xyz="-0.064 0.0245 -0.0265" rpy="0 0.17 ${M_PI}"/>
+    <xacro:generic_camera name="stereo/right" parent="base_link" ros_topic="image_raw" cam_info_topic="camera_info" update_rate="30" res_x="320" res_y="240" image_format="R8G8B8" hfov="65.0">
+      <origin xyz="-0.064 0.0245 -0.0265" rpy="0 0.261 ${M_PI}"/>
     </xacro:generic_camera>
 <!-- TOF camera -->

Commit message: camera placement

File: spiri_description/sensors/quadrotor_sensors.gazebo.xacro (robot description, xacro)
@@ -60,10 +60,10 @@
     <xacro:include filename="$(find spiri_description)/sensors/generic_camera.urdf.xacro" />
     <xacro:generic_camera name="stereo/left" parent="base_link" ros_topic="image_raw" cam_info_topic="camera_info" update_rate="30" res_x="320" res_y="240" image_format="R8G8B8" hfov="65.0">
-      <origin xyz="-0.064 -0.0245 -0.0265" rpy="0 0.261 ${M_PI}"/>
+      <origin xyz="-0.064 -0.0245 -0.0265" rpy="0 0.27 ${M_PI}"/>
     </xacro:generic_camera>
 <!-- Right Forward facing camera -->
     <xacro:include filename="$(find spiri_description)/sensors/generic_camera.urdf.xacro" />
     <xacro:generic_camera name="stereo/right" parent="base_link" ros_topic="image_raw" cam_info_topic="camera_info" update_rate="30" res_x="320" res_y="240" image_format="R8G8B8" hfov="65.0">
-      <origin xyz="-0.064 0.0245 -0.0265" rpy="0 0.261 ${M_PI}"/>
+      <origin xyz="-0.064 0.0245 -0.0265" rpy="0 0.27 ${M_PI}"/>
     </xacro:generic_camera>
 <!-- TOF camera -->

Commit message: fixed the bottom camera - rotated by 180

File: spiri_description/sensors/quadrotor_sensors.gazebo.xacro (robot description, xacro)
@@ -55,5 +55,5 @@
     <xacro:include filename="$(find spiri_description)/sensors/generic_camera.urdf.xacro" />
     <xacro:generic_camera name="downward_cam" parent="base_link" ros_topic="camera/image" cam_info_topic="camera/camera_info" update_rate="30" res_x="640" res_y="480" image_format="R8G8B8" hfov="65">
-      <origin xyz="-0.04 0.0 -0.035" rpy="0 ${M_PI/2} 0"/>
+      <origin xyz="-0.04 0.0 -0.035" rpy="0 ${M_PI/2} ${M_PI}"/>
  </xacro:generic_camera>
 <!-- Left Forward facing camera -->

Commit message: new mesh file

File: spiri_description/sensors/quadrotor_sensors.gazebo.xacro (robot description, xacro)
@@ -55,20 +55,20 @@
     <xacro:include filename="$(find spiri_description)/sensors/generic_camera.urdf.xacro" />
     <xacro:generic_camera name="downward_cam" parent="base_link" ros_topic="camera/image" cam_info_topic="camera/camera_info" update_rate="30" res_x="640" res_y="480" image_format="R8G8B8" hfov="65">
-      <origin xyz="-0.04 0.0 -0.035" rpy="0 ${M_PI/2} ${M_PI}"/>
+      <origin xyz="-0.04 0.0 -0.015" rpy="0 ${M_PI/2} ${M_PI}"/>
  </xacro:generic_camera>
 <!-- Left Forward facing camera -->
     <xacro:include filename="$(find spiri_description)/sensors/generic_camera.urdf.xacro" />
     <xacro:generic_camera name="stereo/left" parent="base_link" ros_topic="image_raw" cam_info_topic="camera_info" update_rate="30" res_x="320" res_y="240" image_format="R8G8B8" hfov="65.0">
-      <origin xyz="-0.064 -0.0245 -0.0265" rpy="0 0.27 ${M_PI}"/>
+      <origin xyz="-0.064 -0.0245 -0.005" rpy="0 0.27 ${M_PI}"/>
     </xacro:generic_camera>
 <!-- Right Forward facing camera -->
     <xacro:include filename="$(find spiri_description)/sensors/generic_camera.urdf.xacro" />
     <xacro:generic_camera name="stereo/right" parent="base_link" ros_topic="image_raw" cam_info_topic="camera_info" update_rate="30" res_x="320" res_y="240" image_format="R8G8B8" hfov="65.0">
-      <origin xyz="-0.064 0.0245 -0.0265" rpy="0 0.27 ${M_PI}"/>
+      <origin xyz="-0.064 0.0245 -0.005" rpy="0 0.27 ${M_PI}"/>
     </xacro:generic_camera>
 <!-- TOF camera -->
  <!--xacro:include filename="$(find spiri_description)/sensors/tof_kinect.urdf.xacro" />
      <xacro:kinect_camera name="camera" parent="base_link">
-      <origin xyz="-0.04 -0.00 0.1" rpy="0 0 ${M_PI}"/>
+      <origin xyz="-0.04 -0.00 0.05" rpy="0 0 ${M_PI}"/>
     </xacro:kinect_camera-->
  <!--xacro:include filename="$(find spiri_description)/sensors/tof.urdf.xacro" />

File: spiri_description/urdf/spiri_base.urdf.xacro (robot description, xacro)
@@ -23,5 +23,5 @@
       <geometry>
         <mesh
-          filename="package://spiri_description/meshes/spiri.STL" />
+          filename="package://spiri_description/meshes/spiri.dae" />
       </geometry>
     </visual>
