Commit message: spiri_api

File: spiri_description/sensors/quadrotor_sensors.gazebo.xacro (robot description, xacro)
@@ -55,20 +55,20 @@
     <xacro:include filename="$(find spiri_description)/sensors/generic_camera.urdf.xacro" />
     <xacro:generic_camera name="downward_cam" parent="base_link" ros_topic="camera/image" cam_info_topic="camera/camera_info" update_rate="30" res_x="640" res_y="480" image_format="R8G8B8" hfov="65">
-      <origin xyz="-0.04 0.0 -0.015" rpy="0 ${M_PI/2} ${M_PI}"/>
+      <origin xyz="-0.04 0.0 -0.035" rpy="0 ${M_PI/2} ${M_PI}"/>
  </xacro:generic_camera>
 <!-- Left Forward facing camera -->
     <xacro:include filename="$(find spiri_description)/sensors/generic_camera.urdf.xacro" />
     <xacro:generic_camera name="stereo/left" parent="base_link" ros_topic="image_raw" cam_info_topic="camera_info" update_rate="30" res_x="320" res_y="240" image_format="R8G8B8" hfov="65.0">
-      <origin xyz="-0.064 -0.0245 -0.005" rpy="0 0.27 ${M_PI}"/>
+      <origin xyz="-0.064 -0.0245 -0.0265" rpy="0 0.27 ${M_PI}"/>
     </xacro:generic_camera>
 <!-- Right Forward facing camera -->
     <xacro:include filename="$(find spiri_description)/sensors/generic_camera.urdf.xacro" />
     <xacro:generic_camera name="stereo/right" parent="base_link" ros_topic="image_raw" cam_info_topic="camera_info" update_rate="30" res_x="320" res_y="240" image_format="R8G8B8" hfov="65.0">
-      <origin xyz="-0.064 0.0245 -0.005" rpy="0 0.27 ${M_PI}"/>
+      <origin xyz="-0.064 0.0245 -0.0265" rpy="0 0.27 ${M_PI}"/>
     </xacro:generic_camera>
 <!-- TOF camera -->
  <!--xacro:include filename="$(find spiri_description)/sensors/tof_kinect.urdf.xacro" />
      <xacro:kinect_camera name="camera" parent="base_link">
-      <origin xyz="-0.04 -0.00 0.05" rpy="0 0 ${M_PI}"/>
+      <origin xyz="-0.04 -0.00 0.1" rpy="0 0 ${M_PI}"/>
     </xacro:kinect_camera-->
  <!--xacro:include filename="$(find spiri_description)/sensors/tof.urdf.xacro" />

Commit message: backup

File: spiri_description/sensors/quadrotor_sensors.gazebo.xacro (robot description, xacro)
@@ -63,8 +63,8 @@
     </xacro:generic_camera>
 <!-- Right Forward facing camera -->
-    <xacro:include filename="$(find spiri_description)/sensors/generic_camera.urdf.xacro" />
+    <!--xacro:include filename="$(find spiri_description)/sensors/generic_camera.urdf.xacro" />
     <xacro:generic_camera name="stereo/right" parent="base_link" ros_topic="image_raw" cam_info_topic="camera_info" update_rate="30" res_x="640" res_y="480" image_format="R8G8B8" hfov="65.0">
       <origin xyz="-0.064 0.0245 -0.0265" rpy="0 0.27 ${M_PI}"/>
-    </xacro:generic_camera>
+    </xacro:generic_camera-->
 <!-- TOF camera -->
  <!--xacro:include filename="$(find spiri_description)/sensors/tof_kinect.urdf.xacro" />
@@ -72,7 +72,7 @@
       <origin xyz="-0.04 -0.00 0.1" rpy="0 0 ${M_PI}"/>
     </xacro:kinect_camera-->
- <!--xacro:include filename="$(find spiri_description)/sensors/tof.urdf.xacro" />
-    <xacro:generic_tof name="tof" parent="forward_cam_link" ros_topic="tof" update_rate="30" noise="0.0">
-      <origin xyz="0.00 0.0 0.02" rpy="${M_PI} 0 0"/>
-    </xacro:generic_tof-->
+ <xacro:include filename="$(find spiri_description)/sensors/tof.urdf.xacro" />
+    <xacro:generic_tof name="tof" parent="base_link" ros_topic="tof" update_rate="30" noise="0.0">
+      <origin xyz="-0.064 0.0 0.2" rpy="0 0 ${M_PI}"/>
+    </xacro:generic_tof>
 </robot>

Commit message: kinect just for collision

File: spiri_description/sensors/quadrotor_sensors.gazebo.xacro (robot description, xacro)
@@ -68,11 +68,11 @@
     </xacro:generic_camera-->
 <!-- TOF camera -->
- <!--xacro:include filename="$(find spiri_description)/sensors/tof_kinect.urdf.xacro" />
+ <xacro:include filename="$(find spiri_description)/sensors/tof_kinect.urdf.xacro" />
      <xacro:kinect_camera name="camera" parent="base_link">
-      <origin xyz="-0.04 -0.00 0.1" rpy="0 0 ${M_PI}"/>
-    </xacro:kinect_camera-->
- <xacro:include filename="$(find spiri_description)/sensors/tof.urdf.xacro" />
+      <origin xyz="-0.064 -0.00 0.2" rpy="0 0 ${M_PI}"/>
+    </xacro:kinect_camera>
+ <!--xacro:include filename="$(find spiri_description)/sensors/tof.urdf.xacro" />
     <xacro:generic_tof name="tof" parent="base_link" ros_topic="tof" update_rate="30" noise="0.0">
       <origin xyz="-0.064 0.0 0.2" rpy="0 0 ${M_PI}"/>
-    </xacro:generic_tof>
+    </xacro:generic_tof-->
 </robot>

Commit message: Making simulated sensors match real sensors

File: spiri_description/sensors/quadrotor_sensors.gazebo.xacro (robot description, xacro)
@@ -1,5 +1,46 @@
 <?xml version="1.0"?>
 <robot xmlns:xacro="http://ros.org/wiki/xacro">
-  <!-- Quadrotor Sensor Plugins -->
+  <xacro:property name="M_PI" value="3.1415926535897931" />
+  <!-- Downward facing camera -->
+  <xacro:include filename="$(find spiri_description)/sensors/generic_camera.urdf.xacro" />
+  <xacro:generic_camera name="downward_cam" parent="base_link" ros_topic="camera/image" cam_info_topic="camera/camera_info" update_rate="30" res_x="640" res_y="480" image_format="R8G8B8" hfov="65">
+    <origin xyz="-0.04 0.0 -0.035" rpy="0 ${M_PI/2} ${M_PI}"/>
+  </xacro:generic_camera>
+  <!-- Left Forward facing camera -->
+  <xacro:generic_camera name="stereo/left" parent="base_link" ros_topic="image_raw" cam_info_topic="camera_info" update_rate="30" res_x="640" res_y="480" image_format="R8G8B8" hfov="65.0">
+    <origin xyz="0.064 0.0245 -0.0265" rpy="0 0.27 0"/>
+  </xacro:generic_camera>
+  <!-- Right Forward facing camera -->
+  <xacro:generic_camera name="stereo/right" parent="base_link" ros_topic="image_raw" cam_info_topic="camera_info" update_rate="30" res_x="640" res_y="480" image_format="R8G8B8" hfov="65.0">
+    <origin xyz="0.064 -0.0245 -0.0265" rpy="0 0.27 0"/>
+  </xacro:generic_camera>
+  <gazebo reference="range_link">
+    <sensor type="ray" name="range">
+      <always_on>true</always_on>
+      <update_rate>100</update_rate>
+      <pose>0 0 0 0 0 0</pose>
+      <visualize>true</visualize>
+      <ray>
+        <scan>
+          <horizontal>
+            <samples>10</samples>
+            <resolution>1</resolution>
+            <min_angle>${-M_PI/20}</min_angle>
+            <max_angle>${M_PI/20}</max_angle>
+          </horizontal>
+        </scan>
+        <range>
+          <min>0.01</min>
+          <max>10</max>
+          <resolution>0.01</resolution>
+        </range>
+      </ray>
+      <plugin name="gazebo_ros_range_controller" filename="libhector_gazebo_ros_sonar.so">
+        <gaussianNoise>0.005</gaussianNoise>
+        <topicName>range</topicName>
+        <frameId>range_link</frameId>
+      </plugin>
+    </sensor>
+  </gazebo>
   <gazebo>
     <plugin name="quadrotor_imu_sim" filename="libhector_gazebo_ros_imu.so">
@@ -15,13 +56,4 @@
       <headingDrift>0.1</headingDrift>
       <headingGaussianNoise>0.05</headingGaussianNoise>
-    </plugin>
-    <plugin name="quadrotor_baro_sim" filename="libhector_gazebo_ros_baro.so">
-      <updateRate>30.0</updateRate>
-      <bodyName>base_link</bodyName>
-      <topicName>pressure_height</topicName>
-      <altimeterTopicName>altimeter</altimeterTopicName>
-      <offset>0</offset>
-      <drift>0.0</drift>
-      <gaussianNoise>0.0</gaussianNoise>
     </plugin>
     <plugin name="quadrotor_magnetic_sim" filename="libhector_gazebo_ros_magnetic.so">
@@ -50,28 +82,3 @@
     </plugin>
 </gazebo>
-   <xacro:property name="M_PI" value="3.1415926535897931" />
-    <!-- Downward facing camera -->
-    <xacro:include filename="$(find spiri_description)/sensors/generic_camera.urdf.xacro" />
-    <xacro:generic_camera name="downward_cam" parent="base_link" ros_topic="camera/image" cam_info_topic="camera/camera_info" update_rate="30" res_x="640" res_y="480" image_format="R8G8B8" hfov="65">
-      <origin xyz="-0.04 0.0 -0.035" rpy="0 ${M_PI/2} ${M_PI}"/>
- </xacro:generic_camera>
-<!-- Left Forward facing camera -->
-    <xacro:include filename="$(find spiri_description)/sensors/generic_camera.urdf.xacro" />
-    <xacro:generic_camera name="stereo/left" parent="base_link" ros_topic="image_raw" cam_info_topic="camera_info" update_rate="30" res_x="640" res_y="480" image_format="R8G8B8" hfov="65.0">
-      <origin xyz="0.064 0.0245 -0.0265" rpy="0 0.27 0"/>
-    </xacro:generic_camera>
-<!-- Right Forward facing camera -->
-    <xacro:include filename="$(find spiri_description)/sensors/generic_camera.urdf.xacro" />
-    <xacro:generic_camera name="stereo/right" parent="base_link" ros_topic="image_raw" cam_info_topic="camera_info" update_rate="30" res_x="640" res_y="480" image_format="R8G8B8" hfov="65.0">
-      <origin xyz="0.064 -0.0245 -0.0265" rpy="0 0.27 0"/>
-    </xacro:generic_camera>
-<!-- TOF camera -->
- <!--xacro:include filename="$(find spiri_description)/sensors/tof_kinect.urdf.xacro" />
-     <xacro:kinect_camera name="camera" parent="base_link">
-      <origin xyz="-0.04 -0.00 0.1" rpy="0 0 ${M_PI}"/>
-    </xacro:kinect_camera-->
- <!--xacro:include filename="$(find spiri_description)/sensors/tof.urdf.xacro" />
-    <xacro:generic_tof name="tof" parent="forward_cam_link" ros_topic="tof" update_rate="30" noise="0.0">
-      <origin xyz="0.00 0.0 0.02" rpy="${M_PI} 0 0"/>
-    </xacro:generic_tof-->
 </robot>

Commit message: Making simulated sensors match real sensors

File: spiri_description/sensors/quadrotor_sensors.gazebo.xacro (robot description, xacro)
@@ -1,5 +1,52 @@
 <?xml version="1.0"?>
 <robot xmlns:xacro="http://ros.org/wiki/xacro">
-  <!-- Quadrotor Sensor Plugins -->
+  <xacro:property name="M_PI" value="3.1415926535897931" />
+  <!-- LINKS FOR ATTACHING SENSORS -->
+  <!-- Downward facing camera -->
+  <xacro:include filename="$(find spiri_description)/sensors/generic_camera.urdf.xacro" />
+  <xacro:generic_camera name="downward_cam" parent="base_link"
+                        ros_topic="camera/image" cam_info_topic="camera/camera_info" update_rate="30"
+                        res_x="640" res_y="480" image_format="R8G8B8" hfov="65" >
+    <origin xyz="-0.04 0.0 -0.035" rpy="0 ${M_PI/2} ${M_PI}"/>
+  </xacro:generic_camera>
+  <!-- Left Forward facing camera -->
+  <xacro:generic_camera name="stereo/left" parent="base_link"
+                        ros_topic="image_raw" cam_info_topic="camera_info" update_rate="30"
+                        res_x="640" res_y="480" image_format="R8G8B8" hfov="65.0">
+    <origin xyz="-0.064 -0.0245 -0.0265" rpy="0 0.27 ${M_PI}"/>
+  </xacro:generic_camera>
+  <xacro:include filename="$(find spiri_description)/sensors/generic_camera.urdf.xacro" />
+    <xacro:generic_camera name="stereo/right" parent="base_link" ros_topic="image_raw" cam_info_topic="camera_info" update_rate="30" res_x="640" res_y="480" image_format="R8G8B8" hfov="65.0">
+    <origin xyz="-0.064 0.0245 -0.0265" rpy="0 0.27 ${M_PI}"/>
+  </xacro:generic_camera>
+  <gazebo reference="range_link">
+    <sensor type="ray" name="range">
+      <always_on>true</always_on>
+      <update_rate>100</update_rate>
+      <pose>0 0 0 0 0 0</pose>
+      <visualize>true</visualize>
+      <ray>
+        <scan>
+          <horizontal>
+            <samples>10</samples>
+            <resolution>1</resolution>
+            <min_angle>${-M_PI/20}</min_angle>
+            <max_angle>${M_PI/20}</max_angle>
+          </horizontal>
+        </scan>
+        <range>
+          <min>0.01</min>
+          <max>10</max>
+          <resolution>0.01</resolution>
+        </range>
+      </ray>
+      <plugin name="gazebo_ros_range_controller" filename="libhector_gazebo_ros_sonar.so">
+        <gaussianNoise>0.005</gaussianNoise>
+        <topicName>range</topicName>
+        <frameId>range_link</frameId>
+      </plugin>
+    </sensor>
+  </gazebo>
+  <!-- SENSOR PLUGINS-->
   <gazebo>
     <plugin name="quadrotor_imu_sim" filename="libhector_gazebo_ros_imu.so">
@@ -15,13 +62,4 @@
       <headingDrift>0.1</headingDrift>
       <headingGaussianNoise>0.05</headingGaussianNoise>
-    </plugin>
-    <plugin name="quadrotor_baro_sim" filename="libhector_gazebo_ros_baro.so">
-      <updateRate>30.0</updateRate>
-      <bodyName>base_link</bodyName>
-      <topicName>pressure_height</topicName>
-      <altimeterTopicName>altimeter</altimeterTopicName>
-      <offset>0</offset>
-      <drift>0.0</drift>
-      <gaussianNoise>0.0</gaussianNoise>
     </plugin>
     <plugin name="quadrotor_magnetic_sim" filename="libhector_gazebo_ros_magnetic.so">
@@ -49,29 +87,4 @@
       <frameName>world</frameName>
     </plugin>
-</gazebo>
-   <xacro:property name="M_PI" value="3.1415926535897931" />
-    <!-- Downward facing camera -->
-    <xacro:include filename="$(find spiri_description)/sensors/generic_camera.urdf.xacro" />
-    <xacro:generic_camera name="downward_cam" parent="base_link" ros_topic="camera/image" cam_info_topic="camera/camera_info" update_rate="30" res_x="640" res_y="480" image_format="R8G8B8" hfov="65">
-      <origin xyz="-0.04 0.0 -0.035" rpy="0 ${M_PI/2} ${M_PI}"/>
- </xacro:generic_camera>
-<!-- Left Forward facing camera -->
-    <xacro:include filename="$(find spiri_description)/sensors/generic_camera.urdf.xacro" />
-    <xacro:generic_camera name="stereo/left" parent="base_link" ros_topic="image_raw" cam_info_topic="camera_info" update_rate="30" res_x="640" res_y="480" image_format="R8G8B8" hfov="65.0">
-      <origin xyz="-0.064 -0.0245 -0.0265" rpy="0 0.27 ${M_PI}"/>
-    </xacro:generic_camera>
-<!-- Right Forward facing camera -->
-    <xacro:include filename="$(find spiri_description)/sensors/generic_camera.urdf.xacro" />
-    <xacro:generic_camera name="stereo/right" parent="base_link" ros_topic="image_raw" cam_info_topic="camera_info" update_rate="30" res_x="640" res_y="480" image_format="R8G8B8" hfov="65.0">
-      <origin xyz="-0.064 0.0245 -0.0265" rpy="0 0.27 ${M_PI}"/>
-    </xacro:generic_camera>
-<!-- TOF camera -->
- <!--xacro:include filename="$(find spiri_description)/sensors/tof_kinect.urdf.xacro" />
-     <xacro:kinect_camera name="camera" parent="base_link">
-      <origin xyz="-0.04 -0.00 0.1" rpy="0 0 ${M_PI}"/>
-    </xacro:kinect_camera-->
- <!--xacro:include filename="$(find spiri_description)/sensors/tof.urdf.xacro" />
-    <xacro:generic_tof name="tof" parent="forward_cam_link" ros_topic="tof" update_rate="30" noise="0.0">
-      <origin xyz="0.00 0.0 0.02" rpy="${M_PI} 0 0"/>
-    </xacro:generic_tof-->
+  </gazebo>
 </robot>

File: spiri_description/urdf/spiri_base.urdf.xacro (robot description, xacro)
@@ -1,10 +1,8 @@
 <?xml version="1.0"?>
-<robot name="spiri">
-  <link
-    name="base_link">
+<robot name="spiri" xmlns:xacro="http://ros.org/wiki/xacro">
+  <xacro:property name="M_PI" value="3.1415926535897931" />
+  <link name="base_link">
     <inertial>
-      <origin
-        xyz="0.0 -0.0 0.0"
-        rpy="0 0 0" />
+      <origin xyz="0.0 -0.0 0.0" rpy="0 0 0" />
       <mass value="0.399875434000126" />
       <inertia
@@ -17,7 +15,5 @@
     </inertial>
     <visual>
-      <origin
-        xyz="0 0 0"
-        rpy="0 0 0" />
+      <origin xyz="0 0 0" rpy="0 0 0" />
       <geometry>
         <mesh filename="package://spiri_description/meshes/spiri.STL" />
@@ -29,7 +25,5 @@
     </visual>
     <collision>
-      <origin
-        xyz="0 0 0"
-        rpy="0 0 0" />
+      <origin xyz="0 0 0" rpy="0 0 0" />
       <geometry>
         <box size="0.33 0.33 0.08" />
@@ -37,3 +31,21 @@
     </collision>
   </link>
+  <joint name="base_imu_joint" type="fixed">
+    <origin xyz="0 0 0" rpy="0 0 0" />
+    <parent link="base_link"/>
+    <child link="imu_link" />
+  </joint>
+  <link name="imu_link" />
+  <joint name="base_range_joint" type="fixed">
+    <origin xyz="0 0 -0.05" rpy="0 ${M_PI/2} 0" />
+    <parent link="base_link"/>
+    <child link="range_link" />
+  </joint>
+  <link name="range_link" />
+  <joint name="base_mag_joint" type="fixed">
+    <origin xyz="0 0 0" rpy="0 0 0" />
+    <parent link="base_link"/>
+    <child link="mag_link" />
+  </joint>
+  <link name="mag_link" />
 </robot>

Commit message: Reversed base mesh origin orientation

File: spiri_description/sensors/quadrotor_sensors.gazebo.xacro (robot description, xacro)
@@ -60,10 +60,10 @@
     <xacro:include filename="$(find spiri_description)/sensors/generic_camera.urdf.xacro" />
     <xacro:generic_camera name="stereo/left" parent="base_link" ros_topic="image_raw" cam_info_topic="camera_info" update_rate="30" res_x="640" res_y="480" image_format="R8G8B8" hfov="65.0">
-      <origin xyz="-0.064 -0.0245 -0.0265" rpy="0 0.27 ${M_PI}"/>
+      <origin xyz="0.064 0.0245 -0.0265" rpy="0 0.27 0"/>
     </xacro:generic_camera>
 <!-- Right Forward facing camera -->
     <xacro:include filename="$(find spiri_description)/sensors/generic_camera.urdf.xacro" />
     <xacro:generic_camera name="stereo/right" parent="base_link" ros_topic="image_raw" cam_info_topic="camera_info" update_rate="30" res_x="640" res_y="480" image_format="R8G8B8" hfov="65.0">
-      <origin xyz="-0.064 0.0245 -0.0265" rpy="0 0.27 ${M_PI}"/>
+      <origin xyz="0.064 -0.0245 -0.0265" rpy="0 0.27 0"/>
     </xacro:generic_camera>
 <!-- TOF camera -->
