Commit message: added pose estimation and teleop code

File: spiri_description/sensors/quadrotor_sensors.gazebo.xacro (robot description, xacro)
@@ -1,8 +1,54 @@
 <?xml version="1.0"?>
 <robot xmlns:xacro="http://ros.org/wiki/xacro">
-  <!-- Quadrotor Sensor Plugins -->
+  <xacro:property name="M_PI" value="3.1415926535897931" />
+  <!-- Downward facing camera -->
+  <xacro:include filename="$(find spiri_description)/sensors/generic_camera.urdf.xacro" />
+  <xacro:generic_camera name="downward_cam" parent="base_link" ros_topic="camera/image" cam_info_topic="camera/camera_info" update_rate="30" res_x="640" res_y="480" image_format="R8G8B8" hfov="65">
+    <origin xyz="-0.04 0.0 -0.035" rpy="0 ${M_PI/2} ${M_PI}"/>
+  </xacro:generic_camera>
+  <!-- Left Forward facing camera -->
+  <xacro:generic_camera name="stereo/left" parent="base_link" ros_topic="image_raw" cam_info_topic="camera_info" update_rate="30" res_x="640" res_y="480" image_format="R8G8B8" hfov="65.0">
+    <origin xyz="0.064 0.0245 -0.0265" rpy="0 0.27 0"/>
+  </xacro:generic_camera>
+  <!-- Right Forward facing camera -->
+  <xacro:generic_camera name="stereo/right" parent="base_link" ros_topic="image_raw" cam_info_topic="camera_info" update_rate="30" res_x="640" res_y="480" image_format="R8G8B8" hfov="65.0">
+    <origin xyz="0.064 -0.0245 -0.0265" rpy="0 0.27 0"/>
+  </xacro:generic_camera>
+<!-- TOF camera -->
+ <xacro:include filename="$(find spiri_description)/sensors/tof_kinect.urdf.xacro" />
+     <xacro:kinect_camera name="camera" parent="base_link">
+      <origin xyz="-0.064 -0.00 0.2" rpy="0 0 ${M_PI}"/>
+    </xacro:kinect_camera>
+  <gazebo reference="range_link">
+    <sensor type="ray" name="range">
+      <always_on>true</always_on>
+      <update_rate>100</update_rate>
+      <pose>0 0 0 0 0 0</pose>
+      <visualize>false</visualize>
+      <ray>
+        <scan>
+          <horizontal>
+            <samples>10</samples>
+            <resolution>1</resolution>
+            <min_angle>${-M_PI/20}</min_angle>
+            <max_angle>${M_PI/20}</max_angle>
+          </horizontal>
+        </scan>
+        <range>
+          <min>0.01</min>
+          <max>10</max>
+          <resolution>0.01</resolution>
+        </range>
+      </ray>
+      <plugin name="gazebo_ros_range_controller" filename="libhector_gazebo_ros_sonar.so">
+        <gaussianNoise>0.0001</gaussianNoise>
+		<topicName>range</topicName>
+        <frameId>range_link</frameId>
+      </plugin>
+    </sensor>
+  </gazebo>
   <gazebo>
     <plugin name="quadrotor_imu_sim" filename="libhector_gazebo_ros_imu.so">
-      <updateRate>30.0</updateRate>
+      <updateRate>100.0</updateRate>
       <bodyName>base_link</bodyName>
       <topicName>raw_imu</topicName>
@@ -15,13 +61,4 @@
       <headingDrift>0.1</headingDrift>
       <headingGaussianNoise>0.05</headingGaussianNoise>
-    </plugin>
-    <plugin name="quadrotor_baro_sim" filename="libhector_gazebo_ros_baro.so">
-      <updateRate>30.0</updateRate>
-      <bodyName>base_link</bodyName>
-      <topicName>pressure_height</topicName>
-      <altimeterTopicName>altimeter</altimeterTopicName>
-      <offset>0</offset>
-      <drift>0.0</drift>
-      <gaussianNoise>0.0</gaussianNoise>
     </plugin>
     <plugin name="quadrotor_magnetic_sim" filename="libhector_gazebo_ros_magnetic.so">
@@ -44,35 +81,18 @@
     </plugin>
     <plugin name="quadrotor_groundtruth_sim" filename="libgazebo_ros_p3d.so">
-      <updateRate>30.0</updateRate>
+      <updateRate>100.0</updateRate>
       <bodyName>base_link</bodyName>
       <topicName>ground_truth/state</topicName>
-      <gaussianNoise>0.0</gaussianNoise>
       <frameName>world</frameName>
     </plugin>
-</gazebo>
-   <xacro:property name="M_PI" value="3.1415926535897931" />
-    <!-- Downward facing camera -->
-    <xacro:include filename="$(find spiri_description)/sensors/generic_camera.urdf.xacro" />
-    <xacro:generic_camera name="downward_cam" parent="base_link" ros_topic="camera/image" cam_info_topic="camera/camera_info" update_rate="30" res_x="640" res_y="480" image_format="R8G8B8" hfov="65">
-      <origin xyz="-0.04 0.0 -0.035" rpy="0 ${M_PI/2} ${M_PI}"/>
- </xacro:generic_camera>
-<!-- Left Forward facing camera -->
-    <xacro:include filename="$(find spiri_description)/sensors/generic_camera.urdf.xacro" />
-    <xacro:generic_camera name="stereo/left" parent="base_link" ros_topic="image_raw" cam_info_topic="camera_info" update_rate="30" res_x="640" res_y="480" image_format="R8G8B8" hfov="65.0">
-      <origin xyz="-0.064 -0.0245 -0.0265" rpy="0 0.27 ${M_PI}"/>
-    </xacro:generic_camera>
-<!-- Right Forward facing camera -->
-    <!--xacro:include filename="$(find spiri_description)/sensors/generic_camera.urdf.xacro" />
-    <xacro:generic_camera name="stereo/right" parent="base_link" ros_topic="image_raw" cam_info_topic="camera_info" update_rate="30" res_x="640" res_y="480" image_format="R8G8B8" hfov="65.0">
-      <origin xyz="-0.064 0.0245 -0.0265" rpy="0 0.27 ${M_PI}"/>
-    </xacro:generic_camera-->
-<!-- TOF camera -->
- <xacro:include filename="$(find spiri_description)/sensors/tof_kinect.urdf.xacro" />
-     <xacro:kinect_camera name="camera" parent="base_link">
-      <origin xyz="-0.064 -0.00 0.2" rpy="0 0 ${M_PI}"/>
-    </xacro:kinect_camera>
- <!--xacro:include filename="$(find spiri_description)/sensors/tof.urdf.xacro" />
-    <xacro:generic_tof name="tof" parent="base_link" ros_topic="tof" update_rate="30" noise="0.0">
-      <origin xyz="-0.064 0.0 0.2" rpy="0 0 ${M_PI}"/>
-    </xacro:generic_tof-->
+    <plugin name="quadrotor_baro_sim" filename="libhector_gazebo_ros_baro.so">
+        <updateRate>30.0</updateRate>
+        <bodyName>base_link</bodyName>
+		<topicName>pressure_height</topicName>
+		<altimeterTopicName>altimeter</altimeterTopicName>
+        <offset>0</offset>
+        <drift>0.0</drift>
+        <gaussianNoise>0.0001</gaussianNoise>
+    </plugin>
+  </gazebo>
 </robot>

File: spiri_description/urdf/quadrotor_plugins.gazebo.xacro (robot description, xacro)
@@ -5,7 +5,7 @@
   <xacro:include filename="$(find hector_quadrotor_gazebo)/urdf/quadrotor_propulsion.gazebo.xacro" />
   <xacro:include filename="$(find hector_quadrotor_gazebo)/urdf/quadrotor_aerodynamics.gazebo.xacro" />
-  <!--xacro:include filename="$(find hector_quadrotor_gazebo)/urdf/quadrotor_rtt_pose_estimation.gazebo.xacro" /-->
-  <!--xacro:include filename="$(find hector_quadrotor_gazebo)/urdf/quadrotor_rtt_controller.gazebo.xacro" /-->
-  <!--xacro:include filename="$(find hector_quadrotor_gazebo)/urdf/quadrotor_rtt_plugin.gazebo.xacro" /-->
+  <!--xacro:include filename="$(find hector_quadrotor_gazebo)/urdf/quadrotor_rtt_pose_estimation.gazebo.xacro" />
+  <xacro:include filename="$(find hector_quadrotor_gazebo)/urdf/quadrotor_rtt_controller.gazebo.xacro" />
+  <xacro:include filename="$(find hector_quadrotor_gazebo)/urdf/quadrotor_rtt_plugin.gazebo.xacro" /-->
   <!-- Quadrotor Gazebo Plugins -->
   <xacro:quadrotor_sensors />

Commit message: Added a stereo camera simulation and tested with collision warning

File: spiri_description/sensors/quadrotor_sensors.gazebo.xacro (robot description, xacro)
@@ -1,97 +1,96 @@
 <?xml version="1.0"?>
 <robot xmlns:xacro="http://ros.org/wiki/xacro">
-  <xacro:property name="M_PI" value="3.1415926535897931" />
-  <!-- Downward facing camera -->
-  <xacro:include filename="$(find spiri_description)/sensors/generic_camera.urdf.xacro" />
-  <xacro:generic_camera name="downward_cam" parent="base_link" ros_topic="camera/image" cam_info_topic="camera/camera_info" update_rate="30" res_x="640" res_y="480" image_format="R8G8B8" hfov="65">
+<xacro:include filename="$(find spiri_description)/sensors/generic_camera.urdf.xacro" />
+<xacro:include filename="$(find spiri_description)/sensors/stereo_camera.urdf.xacro" />
+<xacro:include filename="$(find spiri_description)/sensors/tof_kinect.urdf.xacro" />
+<xacro:property name="M_PI" value="3.1415926535897931" />
+<!-- Downward facing camera -->
+<xacro:generic_camera name="downward_cam" parent="base_link" ros_topic="camera/image" cam_info_topic="camera/camera_info" update_rate="30" res_x="640" res_y="480" image_format="R8G8B8" hfov="65">
     <origin xyz="-0.04 0.0 -0.035" rpy="0 ${M_PI/2} ${M_PI}"/>
-  </xacro:generic_camera>
-  <!-- Left Forward facing camera -->
-  <xacro:generic_camera name="stereo/left" parent="base_link" ros_topic="image_raw" cam_info_topic="camera_info" update_rate="30" res_x="640" res_y="480" image_format="R8G8B8" hfov="65.0">
-    <origin xyz="0.064 0.0245 -0.0265" rpy="0 0.27 0"/>
-  </xacro:generic_camera>
-  <!-- Right Forward facing camera -->
-  <xacro:generic_camera name="stereo/right" parent="base_link" ros_topic="image_raw" cam_info_topic="camera_info" update_rate="30" res_x="640" res_y="480" image_format="R8G8B8" hfov="65.0">
-    <origin xyz="0.064 -0.0245 -0.0265" rpy="0 0.27 0"/>
-  </xacro:generic_camera>
- <xacro:include filename="$(find spiri_description)/sensors/tof_kinect.urdf.xacro" />
-     <xacro:kinect_camera name="camera" parent="base_link">
-      <origin xyz="-0.064 -0.00 0.2" rpy="0 0 ${M_PI}"/>
-    </xacro:kinect_camera>
-  <gazebo reference="range_link">
+</xacro:generic_camera>
+<!-- Stereo camera -->
+<xacro:stereo_camera name="stereo" parent="base_link" baseline="0.049"
+    image_topic="image_raw" cam_info_topic="camera_info" update_rate="30"
+    res_x="640" res_y="480" image_format="R8G8B8" hfov="65.0">
+        <origin xyz="0.064 0 0.0245" rpy="0 0.27 0" />
+</xacro:stereo_camera>
+<xacro:kinect_camera name="camera" parent="base_link">
+    <origin xyz="-0.064 -0.00 0.2" rpy="0 0 ${M_PI}"/>
+</xacro:kinect_camera>
+<gazebo reference="range_link">
     <sensor type="ray" name="range">
-      <always_on>true</always_on>
-      <update_rate>100</update_rate>
-      <pose>0 0 0 0 0 0</pose>
-      <visualize>false</visualize>
-      <ray>
-        <scan>
-          <horizontal>
-            <samples>10</samples>
-            <resolution>1</resolution>
-            <min_angle>${-M_PI/20}</min_angle>
-            <max_angle>${M_PI/20}</max_angle>
-          </horizontal>
-        </scan>
-        <range>
-          <min>0.01</min>
-          <max>10</max>
-          <resolution>0.01</resolution>
-        </range>
-      </ray>
-      <plugin name="gazebo_ros_range_controller" filename="libhector_gazebo_ros_sonar.so">
+        <always_on>true</always_on>
+        <update_rate>100</update_rate>
+        <pose>0 0 0 0 0 0</pose>
+        <visualize>false</visualize>
+        <ray>
+            <scan>
+                <horizontal>
+                    <samples>10</samples>
+                    <resolution>1</resolution>
+                    <min_angle>${-M_PI/20}</min_angle>
+                    <max_angle>${M_PI/20}</max_angle>
+                </horizontal>
+            </scan>
+            <range>
+                <min>0.01</min>
+                <max>10</max>
+                <resolution>0.01</resolution>
+            </range>
+        </ray>
+        <plugin name="gazebo_ros_range_controller" filename="libhector_gazebo_ros_sonar.so">
         <gaussianNoise>0.0001</gaussianNoise>
-		<topicName>range</topicName>
+        <topicName>range</topicName>
         <frameId>range_link</frameId>
-      </plugin>
+        </plugin>
     </sensor>
-  </gazebo>
-  <gazebo>
+</gazebo>
+<gazebo>
     <plugin name="quadrotor_imu_sim" filename="libhector_gazebo_ros_imu.so">
-      <updateRate>100.0</updateRate>
-      <bodyName>base_link</bodyName>
-      <topicName>raw_imu</topicName>
-      <rpyOffsets>0 0 0</rpyOffsets> <!-- deprecated -->
-      <gaussianNoise>0</gaussianNoise>  <!-- deprecated -->
-      <accelDrift>0.5 0.5 0.5</accelDrift>
-      <accelGaussianNoise>0.35 0.35 0.3</accelGaussianNoise>
-      <rateDrift>0.1 0.1 0.1</rateDrift>
-      <rateGaussianNoise>0.05 0.05 0.015</rateGaussianNoise>
-      <headingDrift>0.1</headingDrift>
-      <headingGaussianNoise>0.05</headingGaussianNoise>
+        <updateRate>100.0</updateRate>
+        <bodyName>base_link</bodyName>
+        <topicName>raw_imu</topicName>
+        <rpyOffsets>0 0 0</rpyOffsets> <!-- deprecated -->
+        <gaussianNoise>0</gaussianNoise>  <!-- deprecated -->
+        <accelDrift>0.5 0.5 0.5</accelDrift>
+        <accelGaussianNoise>0.35 0.35 0.3</accelGaussianNoise>
+        <rateDrift>0.1 0.1 0.1</rateDrift>
+        <rateGaussianNoise>0.05 0.05 0.015</rateGaussianNoise>
+        <headingDrift>0.1</headingDrift>
+        <headingGaussianNoise>0.05</headingGaussianNoise>
     </plugin>
     <plugin name="quadrotor_magnetic_sim" filename="libhector_gazebo_ros_magnetic.so">
-      <updateRate>30.0</updateRate>
-      <bodyName>base_link</bodyName>
-      <topicName>magnetic</topicName>
-      <offset>0 0 0</offset>
-      <drift>0.0 0.0 0.0</drift>
-      <gaussianNoise>1.3e-2 1.3e-2 1.3e-2</gaussianNoise>
+        <updateRate>30.0</updateRate>
+        <bodyName>base_link</bodyName>
+        <topicName>magnetic</topicName>
+        <offset>0 0 0</offset>
+        <drift>0.0 0.0 0.0</drift>
+        <gaussianNoise>1.3e-2 1.3e-2 1.3e-2</gaussianNoise>
     </plugin>
     <plugin name="quadrotor_gps_sim" filename="libhector_gazebo_ros_gps.so">
-      <updateRate>30.0</updateRate>
-      <bodyName>base_link</bodyName>
-      <topicName>fix</topicName>
-      <velocityTopicName>fix_velocity</velocityTopicName>
-      <drift>0.0 0.0 0.0</drift>
-      <gaussianNoise>0.01 0.01 0.01</gaussianNoise>
-      <velocityDrift>0 0 0</velocityDrift>
-      <velocityGaussianNoise>0.05 0.05 0.05</velocityGaussianNoise>
+        <updateRate>30.0</updateRate>
+        <bodyName>base_link</bodyName>
+        <topicName>fix</topicName>
+        <velocityTopicName>fix_velocity</velocityTopicName>
+        <drift>0.0 0.0 0.0</drift>
+        <gaussianNoise>0.01 0.01 0.01</gaussianNoise>
+        <velocityDrift>0 0 0</velocityDrift>
+        <velocityGaussianNoise>0.05 0.05 0.05</velocityGaussianNoise>
     </plugin>
     <plugin name="quadrotor_groundtruth_sim" filename="libgazebo_ros_p3d.so">
-      <updateRate>100.0</updateRate>
-      <bodyName>base_link</bodyName>
-      <topicName>ground_truth/state</topicName>
-      <frameName>world</frameName>
+        <updateRate>100.0</updateRate>
+        <bodyName>base_link</bodyName>
+        <topicName>ground_truth/state</topicName>
+        <frameName>world</frameName>
     </plugin>
     <plugin name="quadrotor_baro_sim" filename="libhector_gazebo_ros_baro.so">
         <updateRate>30.0</updateRate>
         <bodyName>base_link</bodyName>
-		<topicName>pressure_height</topicName>
-		<altimeterTopicName>altimeter</altimeterTopicName>
+        <topicName>pressure_height</topicName>
+        <altimeterTopicName>altimeter</altimeterTopicName>
         <offset>0</offset>
         <drift>0.0</drift>
         <gaussianNoise>0.0001</gaussianNoise>
     </plugin>
-  </gazebo>
+</gazebo>
 </robot>

Commit message: Removed kinect simulator

File: spiri_description/sensors/quadrotor_sensors.gazebo.xacro (robot description, xacro)
@@ -15,7 +15,4 @@
         <origin xyz="0.064 0 0.0245" rpy="0 0.27 0" />
 </xacro:stereo_camera>
-<xacro:kinect_camera name="camera" parent="base_link">
-    <origin xyz="-0.064 -0.00 0.2" rpy="0 0 ${M_PI}"/>
-</xacro:kinect_camera>
 <gazebo reference="range_link">
     <sensor type="ray" name="range">

Commit message: changed the position of cameras and fixed action controller

File: spiri_description/sensors/quadrotor_sensors.gazebo.xacro (robot description, xacro)
@@ -3,5 +3,4 @@
 <xacro:include filename="$(find spiri_description)/sensors/generic_camera.urdf.xacro" />
 <xacro:include filename="$(find spiri_description)/sensors/stereo_camera.urdf.xacro" />
-<xacro:include filename="$(find spiri_description)/sensors/tof_kinect.urdf.xacro" />
 <xacro:property name="M_PI" value="3.1415926535897931" />
 <!-- Downward facing camera -->
@@ -13,5 +12,5 @@
     image_topic="image_raw" cam_info_topic="camera_info" update_rate="30"
     res_x="640" res_y="480" image_format="R8G8B8" hfov="65.0">
-        <origin xyz="0.064 0 0.0245" rpy="0 0.27 0" />
+        <origin xyz="0.064 0.0 -0.0265" rpy="0 0.27 0" />
 </xacro:stereo_camera>
 <gazebo reference="range_link">
