Commit message: Revert "Pr 121"

File: spiri_description/sensors/quadrotor_sensors.gazebo.xacro (robot description, xacro)
@@ -1,92 +1,93 @@
 <?xml version="1.0"?>
 <robot xmlns:xacro="http://ros.org/wiki/xacro">
-<xacro:include filename="$(find spiri_description)/sensors/generic_camera.urdf.xacro" />
-<xacro:include filename="$(find spiri_description)/sensors/stereo_camera.urdf.xacro" />
-<xacro:property name="M_PI" value="3.1415926535897931" />
-<!-- Downward facing camera -->
-<xacro:generic_camera name="downward_cam" parent="base_link" ros_topic="camera/image" cam_info_topic="camera/camera_info" update_rate="30" res_x="640" res_y="480" image_format="R8G8B8" hfov="65">
+  <xacro:property name="M_PI" value="3.1415926535897931" />
+  <!-- Downward facing camera -->
+  <xacro:include filename="$(find spiri_description)/sensors/generic_camera.urdf.xacro" />
+  <xacro:generic_camera name="downward_cam" parent="base_link" ros_topic="camera/image" cam_info_topic="camera/camera_info" update_rate="30" res_x="640" res_y="480" image_format="R8G8B8" hfov="65">
     <origin xyz="-0.04 0.0 -0.035" rpy="0 ${M_PI/2} ${M_PI}"/>
-</xacro:generic_camera>
-<!-- Stereo camera -->
-<xacro:stereo_camera name="stereo" parent="base_link" baseline="0.049"
-    image_topic="image_raw" cam_info_topic="camera_info" update_rate="30"
-    res_x="640" res_y="480" image_format="R8G8B8" hfov="65.0">
-        <origin xyz="0.064 0.0 -0.0265" rpy="0 0.27 0" />
-</xacro:stereo_camera>
-<gazebo reference="range_link">
+  </xacro:generic_camera>
+  <!-- Left Forward facing camera -->
+  <xacro:generic_camera name="stereo/left" parent="base_link" ros_topic="image_raw" cam_info_topic="camera_info" update_rate="30" res_x="640" res_y="480" image_format="R8G8B8" hfov="65.0">
+    <origin xyz="0.064 0.0245 -0.0265" rpy="0 0.27 0"/>
+  </xacro:generic_camera>
+  <!-- Right Forward facing camera -->
+  <xacro:generic_camera name="stereo/right" parent="base_link" ros_topic="image_raw" cam_info_topic="camera_info" update_rate="30" res_x="640" res_y="480" image_format="R8G8B8" hfov="65.0">
+    <origin xyz="0.064 -0.0245 -0.0265" rpy="0 0.27 0"/>
+  </xacro:generic_camera>
+  <gazebo reference="range_link">
     <sensor type="ray" name="range">
-        <always_on>true</always_on>
-        <update_rate>100</update_rate>
-        <pose>0 0 0 0 0 0</pose>
-        <visualize>false</visualize>
-        <ray>
-            <scan>
-                <horizontal>
-                    <samples>10</samples>
-                    <resolution>1</resolution>
-                    <min_angle>${-M_PI/20}</min_angle>
-                    <max_angle>${M_PI/20}</max_angle>
-                </horizontal>
-            </scan>
-            <range>
-                <min>0.01</min>
-                <max>10</max>
-                <resolution>0.01</resolution>
-            </range>
-        </ray>
-        <plugin name="gazebo_ros_range_controller" filename="libhector_gazebo_ros_sonar.so">
+      <always_on>true</always_on>
+      <update_rate>100</update_rate>
+      <pose>0 0 0 0 0 0</pose>
+      <visualize>false</visualize>
+      <ray>
+        <scan>
+          <horizontal>
+            <samples>10</samples>
+            <resolution>1</resolution>
+            <min_angle>${-M_PI/20}</min_angle>
+            <max_angle>${M_PI/20}</max_angle>
+          </horizontal>
+        </scan>
+        <range>
+          <min>0.01</min>
+          <max>10</max>
+          <resolution>0.01</resolution>
+        </range>
+      </ray>
+      <plugin name="gazebo_ros_range_controller" filename="libhector_gazebo_ros_sonar.so">
         <gaussianNoise>0.0001</gaussianNoise>
-        <topicName>range</topicName>
+		<topicName>range</topicName>
         <frameId>range_link</frameId>
-        </plugin>
+      </plugin>
     </sensor>
-</gazebo>
-<gazebo>
+  </gazebo>
+  <gazebo>
     <plugin name="quadrotor_imu_sim" filename="libhector_gazebo_ros_imu.so">
-        <updateRate>100.0</updateRate>
-        <bodyName>base_link</bodyName>
-        <topicName>raw_imu</topicName>
-        <rpyOffsets>0 0 0</rpyOffsets> <!-- deprecated -->
-        <gaussianNoise>0</gaussianNoise>  <!-- deprecated -->
-        <accelDrift>0.5 0.5 0.5</accelDrift>
-        <accelGaussianNoise>0.35 0.35 0.3</accelGaussianNoise>
-        <rateDrift>0.1 0.1 0.1</rateDrift>
-        <rateGaussianNoise>0.05 0.05 0.015</rateGaussianNoise>
-        <headingDrift>0.1</headingDrift>
-        <headingGaussianNoise>0.05</headingGaussianNoise>
+      <updateRate>100.0</updateRate>
+      <bodyName>base_link</bodyName>
+      <topicName>raw_imu</topicName>
+      <rpyOffsets>0 0 0</rpyOffsets> <!-- deprecated -->
+      <gaussianNoise>0</gaussianNoise>  <!-- deprecated -->
+      <accelDrift>0.5 0.5 0.5</accelDrift>
+      <accelGaussianNoise>0.35 0.35 0.3</accelGaussianNoise>
+      <rateDrift>0.1 0.1 0.1</rateDrift>
+      <rateGaussianNoise>0.05 0.05 0.015</rateGaussianNoise>
+      <headingDrift>0.1</headingDrift>
+      <headingGaussianNoise>0.05</headingGaussianNoise>
     </plugin>
     <plugin name="quadrotor_magnetic_sim" filename="libhector_gazebo_ros_magnetic.so">
-        <updateRate>30.0</updateRate>
-        <bodyName>base_link</bodyName>
-        <topicName>magnetic</topicName>
-        <offset>0 0 0</offset>
-        <drift>0.0 0.0 0.0</drift>
-        <gaussianNoise>1.3e-2 1.3e-2 1.3e-2</gaussianNoise>
+      <updateRate>30.0</updateRate>
+      <bodyName>base_link</bodyName>
+      <topicName>magnetic</topicName>
+      <offset>0 0 0</offset>
+      <drift>0.0 0.0 0.0</drift>
+      <gaussianNoise>1.3e-2 1.3e-2 1.3e-2</gaussianNoise>
     </plugin>
     <plugin name="quadrotor_gps_sim" filename="libhector_gazebo_ros_gps.so">
-        <updateRate>30.0</updateRate>
-        <bodyName>base_link</bodyName>
-        <topicName>fix</topicName>
-        <velocityTopicName>fix_velocity</velocityTopicName>
-        <drift>0.0 0.0 0.0</drift>
-        <gaussianNoise>0.01 0.01 0.01</gaussianNoise>
-        <velocityDrift>0 0 0</velocityDrift>
-        <velocityGaussianNoise>0.05 0.05 0.05</velocityGaussianNoise>
+      <updateRate>30.0</updateRate>
+      <bodyName>base_link</bodyName>
+      <topicName>fix</topicName>
+      <velocityTopicName>fix_velocity</velocityTopicName>
+      <drift>0.0 0.0 0.0</drift>
+      <gaussianNoise>0.01 0.01 0.01</gaussianNoise>
+      <velocityDrift>0 0 0</velocityDrift>
+      <velocityGaussianNoise>0.05 0.05 0.05</velocityGaussianNoise>
     </plugin>
     <plugin name="quadrotor_groundtruth_sim" filename="libgazebo_ros_p3d.so">
-        <updateRate>100.0</updateRate>
-        <bodyName>base_link</bodyName>
-        <topicName>ground_truth/state</topicName>
-        <frameName>world</frameName>
+      <updateRate>200.0</updateRate>
+      <bodyName>base_link</bodyName>
+      <topicName>ground_truth/state</topicName>
+      <frameName>world</frameName>
     </plugin>
     <plugin name="quadrotor_baro_sim" filename="libhector_gazebo_ros_baro.so">
         <updateRate>30.0</updateRate>
         <bodyName>base_link</bodyName>
-        <topicName>pressure_height</topicName>
-        <altimeterTopicName>altimeter</altimeterTopicName>
+		<topicName>pressure_height</topicName>
+		<altimeterTopicName>altimeter</altimeterTopicName>
         <offset>0</offset>
         <drift>0.0</drift>
         <gaussianNoise>0.0001</gaussianNoise>
     </plugin>
-</gazebo>
+  </gazebo>
 </robot>

File: spiri_description/sensors/tof_kinect.urdf.xacro (robot description, xacro)
@@ -57,11 +57,11 @@
       <gazebo reference="${name}_depth_frame">
         <sensor type="depth" name="${name}">
-          <update_rate>7</update_rate>
+          <update_rate>30</update_rate>
           <camera>
             <horizontal_fov>1.407</horizontal_fov>
             <image>
               <format>R8G8B8</format>
-              <width>320</width>
-              <height>240</height>
+              <width>640</width>
+              <height>480</height>
             </image>
             <clip>
@@ -73,5 +73,5 @@
 	<baseline>0.2</baseline>
 	<alwaysOn>true</alwaysOn>
-            <updateRate>7</updateRate>
+            <updateRate>20</updateRate>
             <imageTopicName>${name}/rgb/image_raw</imageTopicName>
             <cameraInfoTopicName>${name}/rgb/camera_info</cameraInfoTopicName>

Commit message: added new mesh file for Spiri

File: spiri_description/sensors/quadrotor_sensors.gazebo.xacro (robot description, xacro)
@@ -6,5 +6,5 @@
 <!-- Downward facing camera -->
 <xacro:generic_camera name="downward_cam" parent="base_link" ros_topic="camera/image" cam_info_topic="camera/camera_info" update_rate="30" res_x="640" res_y="480" image_format="R8G8B8" hfov="65">
-    <origin xyz="-0.04 0.0 -0.035" rpy="0 ${M_PI/2} ${M_PI}"/>
+    <origin xyz="-0.004 0.070 -0.035" rpy="0 ${M_PI/2} ${M_PI}"/>
 </xacro:generic_camera>
 <!-- Stereo camera -->
@@ -12,5 +12,5 @@
     image_topic="image_raw" cam_info_topic="camera_info" update_rate="30"
     res_x="640" res_y="480" image_format="R8G8B8" hfov="65.0">
-        <origin xyz="0.064 0.0 -0.0265" rpy="0 0.27 0" />
+        <origin xyz="-0.005 0.090 -0.0165" rpy="0 0.34 1.57" />
 </xacro:stereo_camera>
 <gazebo reference="range_link">

File: spiri_description/sensors/stereo_camera.urdf.xacro (robot description, xacro)
@@ -25,5 +25,5 @@
             <origin xyz="0 0 0" rpy="0 0 0" />
             <geometry>
-                <box size="0.005 0.005 0.005" />
+                <box size="0.001 0.001 0.001" />
             </geometry>
             <material name="Blue">
@@ -34,5 +34,5 @@
             <origin xyz="0 0 0" rpy="0 0 0" />
             <geometry>
-                <box size="0.01 0.01 0.01" />
+                <box size="0.001 0.001 0.001" />
             </geometry>
         </collision>
@@ -52,5 +52,5 @@
             <origin xyz="0 0 0" rpy="0 0 0" />
             <geometry>
-                <box size="0.01 0.01 0.01" />
+                <box size="0.001 0.001 0.001" />
             </geometry>
             <material name="Red">
@@ -61,5 +61,5 @@
             <origin xyz="0 0 0" rpy="0 0 0" />
             <geometry>
-                <box size="0.01 0.01 0.01" />
+                <box size="0.001 0.001 0.001" />
             </geometry>
         </collision>
@@ -79,5 +79,5 @@
             <origin xyz="0 0 0" rpy="0 0 0" />
             <geometry>
-                <box size="0.01 0.01 0.01" />
+                <box size="0.001 0.001 0.001" />
             </geometry>
             <material name="Red">
@@ -88,5 +88,5 @@
             <origin xyz="0 0 0" rpy="0 0 0" />
             <geometry>
-                <box size="0.01 0.01 0.01" />
+                <box size="0.001 0.001 0.001" />
             </geometry>
         </collision>

File: spiri_description/urdf/spiri_base.urdf.xacro (robot description, xacro)
@@ -17,5 +17,5 @@
       <origin xyz="0 0 0" rpy="0 0 0" />
       <geometry>
-        <mesh filename="package://spiri_description/meshes/spiri.STL" />
+        <mesh filename="package://spiri_description/meshes/spiri.dae" />
       </geometry>
       <!-- This sets the color in rviz, but not gazebo -->
@@ -32,5 +32,5 @@
  </link>
  <gazebo reference="base_link">
-	 <material>Gazebo/White</material>
+	 <!--material>Gazebo/White</material-->
 	 <turnGravityOff>false</turnGravityOff>
  </gazebo>

Commit message: fixed wrong axis

File: spiri_description/sensors/quadrotor_sensors.gazebo.xacro (robot description, xacro)
@@ -6,5 +6,5 @@
 <!-- Downward facing camera -->
 <xacro:generic_camera name="downward_cam" parent="base_link" ros_topic="camera/image" cam_info_topic="camera/camera_info" update_rate="30" res_x="640" res_y="480" image_format="R8G8B8" hfov="65">
-    <origin xyz="-0.004 0.070 -0.035" rpy="0 ${M_PI/2} ${M_PI}"/>
+    <origin xyz="0.070 0.004 -0.035" rpy="0 ${M_PI/2} ${M_PI}"/>
 </xacro:generic_camera>
 <!-- Stereo camera -->
@@ -12,5 +12,5 @@
     image_topic="image_raw" cam_info_topic="camera_info" update_rate="30"
     res_x="640" res_y="480" image_format="R8G8B8" hfov="65.0">
-        <origin xyz="-0.005 0.090 -0.0165" rpy="0 0.34 1.57" />
+        <origin xyz="0.080 0.005 -0.0165" rpy="0 0.34 0" />
 </xacro:stereo_camera>
 <gazebo reference="range_link">

File: spiri_description/sensors/stereo_camera.urdf.xacro (robot description, xacro)
@@ -34,5 +34,5 @@
             <origin xyz="0 0 0" rpy="0 0 0" />
             <geometry>
-                <box size="0.001 0.001 0.001" />
+                <box size="0.01 0.01 0.01" />
             </geometry>
         </collision>

File: spiri_description/urdf/spiri_base.urdf.xacro (robot description, xacro)
@@ -15,5 +15,5 @@
     </inertial>
     <visual>
-      <origin xyz="0 0 0" rpy="0 0 0" />
+      <origin xyz="0 0 0" rpy="0 0 -1.57" />
       <geometry>
         <mesh filename="package://spiri_description/meshes/spiri.dae" />
