Commit message: move it files for spiri

File: spiri_description/urdf/spiri_base.urdf.xacro (robot description, xacro)
@@ -5,5 +5,5 @@
     <inertial>
       <origin
-        xyz="0.0 -0.0 -0.0"
+        xyz="0.0 -0.0 0.0"
         rpy="0 0 0" />
       <mass
@@ -25,9 +25,4 @@
           filename="package://spiri_description/meshes/base_link.STL" />
       </geometry>
-      <material
-        name="">
-        <color
-          rgba="1 1 1 1" />
-      </material>
     </visual>
     <collision>

Commit message: Added simplified collision model and colored RobotModel for rviz

File: spiri_description/urdf/spiri_base.urdf.xacro (robot description, xacro)
@@ -7,6 +7,5 @@
         xyz="0.0 -0.0 0.0"
         rpy="0 0 0" />
-      <mass
-        value="0.399875434000126" />
+      <mass value="0.399875434000126" />
       <inertia
         ixx="0.00346570293331384"
@@ -22,7 +21,10 @@
         rpy="0 0 0" />
       <geometry>
-        <mesh
-          filename="package://spiri_description/meshes/spiri.STL" />
+        <mesh filename="package://spiri_description/meshes/spiri.STL" />
       </geometry>
+      <!-- This sets the color in rviz, but not gazebo -->
+      <material name="SpiriWhite">
+        <color rgba="0.8 0.8 0.9 1.0"/>
+      </material>
     </visual>
     <collision>
@@ -31,6 +33,5 @@
         rpy="0 0 0" />
       <geometry>
-        <mesh
-          filename="package://spiri_description/meshes/spiri.STL" />
+        <box size="0.33 0.33 0.08" />
       </geometry>
     </collision>
