Commit message: Fixed coloring in gazebo

File: spiri_description/urdf/spiri.gazebo.xacro (robot description, xacro)
@@ -1,5 +1,5 @@
 <?xml version="1.0"?>
 <robot name="spiri" xmlns:xacro="http://ros.org/wiki/xacro">
-    <xacro:include filename="$(find spiri_description)/urdf/spiri_base.urdf.xacro" />
+	<xacro:include filename="$(find spiri_description)/urdf/spiri_base.urdf.xacro" />
     <xacro:include filename="$(find spiri_description)/urdf/quadrotor_plugins.gazebo.xacro" />
 </robot>

File: spiri_description/urdf/spiri_base.urdf.xacro (robot description, xacro)
@@ -30,5 +30,9 @@
       </geometry>
     </collision>
-  </link>
+ </link>
+ <gazebo reference="base_link">
+	 <material>Gazebo/White</material>
+	 <turnGravityOff>false</turnGravityOff>
+ </gazebo>
   <joint name="base_imu_joint" type="fixed">
     <origin xyz="0 0 0" rpy="0 0 0" />
